Commit message: actualizacion modelo 15/12/15

File: r3cpg_description/urdf/body.urdf.xacro (robot description, xacro)
@@ -2,6 +2,6 @@
 <robot
   xmlns:xacro="http://www.ros.org/wiki/xacro"
-  name="r3cpg_body">
-  <xacro:macro name="body">
+  name="r3cpg_body"  >
+  <xacro:macro name="body" >
     <link
       name="base_link">
@@ -40,21 +40,22 @@
       </collision>
     </link>
-    <link
-      name="leg_base_fr" />
-    <joint
-      name="leg_base_fr_fixed"
+<xacro:macro name="leg" params="prefix1 prefix2 prefix3 prefix4 prefix5 prefix6 prefix7 reflect x y z">
+    <link
+      name="${prefix1}_base" />
+    <joint
+      name="${prefix1}_base_fixed"
       type="fixed">
       <origin
-        xyz="0.121 -0.079 -0.0361"
+        xyz="${0.121*x} ${0.079*y} ${0.0361*z}"
         rpy="0 0 0" />
       <parent
         link="base_link" />
       <child
-        link="leg_base_fr" />
+        link="${prefix1}_base" />
       <axis
         xyz="0 0 0" />
     </joint>
     <link
-      name="leg_shoulder">
+      name="${prefix2}_1">
       <inertial>
         <origin
@@ -92,13 +93,13 @@
     </link>
     <joint
-      name="leg_shoulder_joint"
+      name="${prefix5}_1"
       type="revolute">
       <origin
         xyz="0 -0.00252 0"
-        rpy="0 0 0" />
-      <parent
-        link="leg_base_fr" />
-      <child
-        link="leg_shoulder" />
+        rpy="0 0 ${3.14*(reflect-1.0)/2.0}" />
+      <parent
+        link="${prefix1}_base" />
+      <child
+        link="${prefix2}_1" />
       <axis
         xyz="0 -1 0" />
@@ -110,5 +111,5 @@
     </joint>
     <link
-      name="leg_elbow">
+      name="${prefix3}_2">
       <inertial>
         <origin
@@ -146,5 +147,5 @@
     </link>
     <joint
-      name="leg_elbow_joint"
+      name="${prefix6}_2"
       type="revolute">
       <origin
@@ -152,7 +153,7 @@
         rpy="0 0 0" />
       <parent
-        link="leg_shoulder" />
-      <child
-        link="leg_elbow" />
+        link="${prefix2}_1" />
+      <child
+        link="${prefix3}_2" />
       <axis
         xyz="0 -1 0" />
@@ -164,5 +165,5 @@
     </joint>
     <link
-      name="leg_wrist">
+      name="${prefix4}_3">
       <inertial>
         <origin
@@ -200,5 +201,5 @@
     </link>
     <joint
-      name="leg_wrist_joint"
+      name="${prefix7}_3"
       type="revolute">
       <origin
@@ -206,7 +207,7 @@
         rpy="0 0 0" />
       <parent
-        link="leg_elbow" />
-      <child
-        link="leg_wrist" />
+        link="${prefix3}_2" />
+      <child
+        link="${prefix4}_3" />
       <axis
         xyz="0 -1 0" />
@@ -217,49 +218,9 @@
         velocity="0" />
     </joint>
-    <link
-      name="leg_base_fl" />
-    <joint
-      name="leg_base_fl_fixed"
-      type="fixed">
-      <origin
-        xyz="0.121 0.079 -0.0361"
-        rpy="0 0 0" />
-      <parent
-        link="base_link" />
-      <child
-        link="leg_base_fl" />
-      <axis
-        xyz="0 0 0" />
-    </joint>
-    <link
-      name="leg_base_rr" />
-    <joint
-      name="leg_base_rr_fixed"
-      type="fixed">
-      <origin
-        xyz="-0.121 -0.079 -0.0361"
-        rpy="0 0 0" />
-      <parent
-        link="base_link" />
-      <child
-        link="leg_base_rr" />
-      <axis
-        xyz="0 0 0" />
-    </joint>
-    <link
-      name="leg_base_rl" />
-    <joint
-      name="leg_base_rl_fixed"
-      type="fixed">
-      <origin
-        xyz="-0.121 0.079 -0.0361"
-        rpy="0 0 0" />
-      <parent
-        link="base_link" />
-      <child
-        link="leg_base_rl" />
-      <axis
-        xyz="0 0 0" />
-    </joint>
-  </xacro:macro>
+</xacro:macro>
+<xacro:leg prefix1="leg_fr" prefix2="leg_shoulder_fr" prefix3="leg_elbow_fr" prefix4="leg_wrist_fr" prefix5="leg_shoulder_joint_fr" prefix6="leg_elbow_joint_fr" prefix7="leg_wrist_joint_fr" reflect="1.0" x="1.0" y="-1.0" z="-1.0"/>
+<xacro:leg prefix1="leg_fl" prefix2="leg_shoulder_fl" prefix3="leg_elbow_fl" prefix4="leg_wrist_fl" prefix5="leg_shoulder_joint_fl" prefix6="leg_elbow_joint_fl" prefix7="leg_wrist_joint_fl" reflect="-1.0" x="1.0" y="1.0" z="-1.0"/>
+<xacro:leg prefix1="leg_rr" prefix2="leg_shoulder_rr" prefix3="leg_elbow_rr" prefix4="leg_wrist_rr" prefix5="leg_shoulder_joint_rr" prefix6="leg_elbow_joint_rr" prefix7="leg_wrist_joint_rr" reflect="1.0" x="-1.0" y="-1.0" z="-1.0"/>
+<xacro:leg prefix1="leg_rl" prefix2="leg_shoulder_rl" prefix3="leg_elbow_rl" prefix4="leg_wrist_rl" prefix5="leg_shoulder_joint_rl" prefix6="leg_elbow_joint_rl" prefix7="leg_wrist_joint_rl" reflect="-1.0" x="-1.0" y="1.0" z="-1.0"/>
+</xacro:macro>
 </robot>

Commit message: rama de desarrollo para indigo

File: r3cpg_description/urdf/body.urdf.xacro (robot description, xacro)
@@ -2,6 +2,6 @@
 <robot
   xmlns:xacro="http://www.ros.org/wiki/xacro"
-  name="r3cpg_body"  >
-  <xacro:macro name="body" >
+  name="r3cpg_body">
+  <xacro:macro name="body">
     <link
       name="base_link">
@@ -40,187 +40,64 @@
       </collision>
     </link>
-<xacro:macro name="leg" params="prefix1 prefix2 prefix3 prefix4 prefix5 prefix6 prefix7 reflect x y z">
     <link
-      name="${prefix1}_base" />
+      name="leg_base_fr" />
     <joint
-      name="${prefix1}_base_fixed"
+      name="leg_base_fr_fixed"
       type="fixed">
       <origin
-        xyz="${0.121*x} ${0.079*y} ${0.0361*z}"
+        xyz="0.121 -0.079 -0.0361"
         rpy="0 0 0" />
       <parent
         link="base_link" />
       <child
-        link="${prefix1}_base" />
+        link="leg_base_fr" />
       <axis
         xyz="0 0 0" />
     </joint>
     <link
-      name="${prefix2}_1">
-      <inertial>
-        <origin
-          xyz="1.7689E-08 0.024508 -0.063634"
-          rpy="0 0 0" />
-        <mass
-          value="0.12155" />
-        <inertia
-          ixx="0.0001766"
-          ixy="-3.1201E-11"
-          ixz="-5.9479E-11"
-          iyy="0.00014384"
-          iyz="1.3321E-06"
-          izz="5.9298E-05" />
-      </inertial>
-      <visual>
-        <origin
-          xyz="0 0 0"
-          rpy="0 0 0" />
-        <geometry>
-          <mesh
-            filename="package://r3cpg_description/meshes/leg_shoulder.stl" />
-        </geometry>
-        <material name="Grey1" />
-      </visual>
-      <collision>
-        <origin
-          xyz="0 0 0"
-          rpy="0 0 0" />
-        <geometry>
-          <mesh
-            filename="package://r3cpg_description/meshes/leg_shoulder.stl" />
-        </geometry>
-      </collision>
-    </link>
+      name="leg_base_fl" />
     <joint
-      name="${prefix5}_1"
-      type="revolute">
+      name="leg_base_fl_fixed"
+      type="fixed">
       <origin
-        xyz="0 -0.00252 0"
-        rpy="0 0 ${3.14*(reflect-1.0)/2.0}" />
+        xyz="0.121 0.079 -0.0361"
+        rpy="0 0 0" />
       <parent
-        link="${prefix1}_base" />
+        link="base_link" />
       <child
-        link="${prefix2}_1" />
+        link="leg_base_fl" />
       <axis
-        xyz="0 -1 0" />
-      <limit
-        lower="-1.0"
-        upper="1.0"
-        effort="0"
-        velocity="0" />
+        xyz="0 0 0" />
     </joint>
     <link
-      name="${prefix3}_2">
-      <inertial>
-        <origin
-          xyz="-1.7313E-08 0.026803 -0.063159"
-          rpy="0 0 0" />
-        <mass
-          value="0.12414" />
-        <inertia
-          ixx="0.00018537"
-          ixy="-3.1359E-11"
-          ixz="6.0464E-11"
-          iyy="0.00014551"
-          iyz="-2.1303E-06"
-          izz="6.7084E-05" />
-      </inertial>
-      <visual>
-        <origin
-          xyz="0 0 0"
-          rpy="0 0 0" />
-        <geometry>
-          <mesh
-            filename="package://r3cpg_description/meshes/leg_elbow.stl" />
-        </geometry>
-        <material name="Grey2" />
-      </visual>
-      <collision>
-        <origin
-          xyz="0 0 0"
-          rpy="0 0 0" />
-        <geometry>
-          <mesh
-            filename="package://r3cpg_description/meshes/leg_elbow.stl" />
-        </geometry>
-      </collision>
-    </link>
+      name="leg_base_rr" />
     <joint
-      name="${prefix6}_2"
-      type="revolute">
+      name="leg_base_rr_fixed"
+      type="fixed">
       <origin
-        xyz="0 0.00142 -0.09284"
+        xyz="-0.121 -0.079 -0.0361"
         rpy="0 0 0" />
       <parent
-        link="${prefix2}_1" />
+        link="base_link" />
       <child
-        link="${prefix3}_2" />
+        link="leg_base_rr" />
       <axis
-        xyz="0 -1 0" />
-      <limit
-        lower="-1.0"
-        upper="1.0"
-        effort="0"
-        velocity="0" />
+        xyz="0 0 0" />
     </joint>
     <link
-      name="${prefix4}_3">
-      <inertial>
-        <origin
-          xyz="-4.1233E-10 0.027507 -0.036847"
-          rpy="0 0 0" />
-        <mass
-          value="0.066391" />
-        <inertia
-          ixx="5.2481E-05"
-          ixy="4.1851E-12"
-          ixz="1.8037E-11"
-          iyy="3.0101E-05"
-          iyz="1.7364E-08"
-          izz="3.9757E-05" />
-      </inertial>
-      <visual>
-        <origin
-          xyz="0 0 0"
-          rpy="0 0 0" />
-        <geometry>
-          <mesh
-            filename="package://r3cpg_description/meshes/leg_wrist.stl" />
-        </geometry>
-        <material name="Grey3" />
-      </visual>
-      <collision>
-        <origin
-          xyz="0 0 0"
-          rpy="0 0 0" />
-        <geometry>
-          <mesh
-            filename="package://r3cpg_description/meshes/leg_wrist.stl" />
-        </geometry>
-      </collision>
-    </link>
+      name="leg_base_rl" />
     <joint
-      name="${prefix7}_3"
-      type="revolute">
+      name="leg_base_rl_fixed"
+      type="fixed">
       <origin
-        xyz="0 -0.00092 -0.09284"
+        xyz="-0.121 0.079 -0.0361"
         rpy="0 0 0" />
       <parent
-        link="${prefix3}_2" />
+        link="base_link" />
       <child
-        link="${prefix4}_3" />
+        link="leg_base_rl" />
       <axis
-        xyz="0 -1 0" />
-      <limit
-        lower="-1.0"
-        upper="1.0"
-        effort="0"
-        velocity="0" />
+        xyz="0 0 0" />
     </joint>
-</xacro:macro>
-<xacro:leg prefix1="leg_fr" prefix2="leg_shoulder_fr" prefix3="leg_elbow_fr" prefix4="leg_wrist_fr" prefix5="leg_shoulder_joint_fr" prefix6="leg_elbow_joint_fr" prefix7="leg_wrist_joint_fr" reflect="1.0" x="1.0" y="-1.0" z="-1.0"/>
-<xacro:leg prefix1="leg_fl" prefix2="leg_shoulder_fl" prefix3="leg_elbow_fl" prefix4="leg_wrist_fl" prefix5="leg_shoulder_joint_fl" prefix6="leg_elbow_joint_fl" prefix7="leg_wrist_joint_fl" reflect="-1.0" x="1.0" y="1.0" z="-1.0"/>
-<xacro:leg prefix1="leg_rr" prefix2="leg_shoulder_rr" prefix3="leg_elbow_rr" prefix4="leg_wrist_rr" prefix5="leg_shoulder_joint_rr" prefix6="leg_elbow_joint_rr" prefix7="leg_wrist_joint_rr" reflect="1.0" x="-1.0" y="-1.0" z="-1.0"/>
-<xacro:leg prefix1="leg_rl" prefix2="leg_shoulder_rl" prefix3="leg_elbow_rl" prefix4="leg_wrist_rl" prefix5="leg_shoulder_joint_rl" prefix6="leg_elbow_joint_rl" prefix7="leg_wrist_joint_rl" reflect="-1.0" x="-1.0" y="1.0" z="-1.0"/>
-</xacro:macro>
+  </xacro:macro>
 </robot>
