Commit message: parametros piernas ok

File: r3cpg_description/robots/r3cpg.urdf.xacro (robot description, xacro)
@@ -14,4 +14,9 @@
   <xacro:body/>
   <!-- Legs -->
+  <xacro:include filename="$(find r3cpg_description)/urdf/leg.urdf.xacro" />
+  <xacro:leg  parent="leg_base_rr" side="rr" reflect="1" />
+  <xacro:leg  parent="leg_base_fr" side="fr" reflect="1" />
+  <xacro:leg  parent="leg_base_rl" side="rl" reflect="-1" />
+  <xacro:leg  parent="leg_base_fl" side="fl" reflect="-1" />
   <!-- TODO -->
 </robot>

File: r3cpg_description/urdf/leg.urdf.xacro (robot description, xacro)
@@ -3,7 +3,7 @@
   xmlns:xacro="http://www.ros.org/wiki/xacro"
   name="r3cpg_body"  >
-  <xacro:macro name="leg" params="parent side reflect x y z">
+  <xacro:macro name="leg" params="parent side reflect">
     <link
-      name="leg_shoulder">
+      name="leg_${side}_shoulder">
       <inertial>
         <origin
@@ -41,15 +41,15 @@
     </link>
     <joint
-      name="leg_shoulder_joint"
+      name="leg_${side}_shoulder"
       type="revolute">
       <origin
-        xyz="0 -0.00252 0"
-        rpy="0 0 0" />
+        xyz="0 ${-reflect*0.00252} 0"
+        rpy="0 0 ${(reflect-1.0)/2.0*3.1415}" /><!--  -->
       <parent
         link="${parent}" />
       <child
-        link="leg_shoulder" />
+        link="leg_${side}_shoulder" />
       <axis
-        xyz="0 -1 0" />
+        xyz="0 ${-reflect} 0" />
       <limit
         lower="-1.0"
@@ -59,5 +59,5 @@
     </joint>
     <link
-      name="leg_elbow">
+      name="leg_${side}_elbow">
       <inertial>
         <origin
@@ -95,5 +95,5 @@
     </link>
     <joint
-      name="leg_elbow_joint"
+      name="leg_${side}_elbow_joint"
       type="revolute">
       <origin
@@ -101,9 +101,9 @@
         rpy="0 0 0" />
       <parent
-        link="leg_shoulder" />
+        link="leg_${side}_shoulder" />
       <child
-        link="leg_elbow" />
+        link="leg_${side}_elbow" />
       <axis
-        xyz="0 -1 0" />
+        xyz="0 ${-reflect} 0" />
       <limit
         lower="-1.0"
@@ -113,5 +113,5 @@
     </joint>
     <link
-      name="leg_wrist">
+      name="leg_${side}_wrist">
       <inertial>
         <origin
@@ -149,5 +149,5 @@
     </link>
     <joint
-      name="leg_wrist_joint"
+      name="leg_${side}_wrist_joint"
       type="revolute">
       <origin
@@ -155,9 +155,9 @@
         rpy="0 0 0" />
       <parent
-        link="leg_elbow" />
+        link="leg_${side}_elbow" />
       <child
-        link="leg_wrist" />
+        link="leg_${side}_wrist" />
       <axis
-        xyz="0 -1 0" />
+        xyz="0 ${-reflect} 0" />
       <limit
         lower="-1.0"
